File: KiCad/UserInterface.kicad_sch (KiCad schematic)
At the start: 5 parts, among them J3 LCD_Conn, J4 Enc_Conn, J6 Btn&Led, J7 PWR, J9 Btn_Matrix

Commit message: PCB design
Parts:
- renumbered J9 to J3, J3 to J4, J4 to J5
Changed lines of the file:
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@@
 		(dnp no)
 		(fields_autoplaced yes)
-		(property "Reference" "J3"
+		(property "Reference" "J4"
 			(at 49.53 113.0299 0)
 			(effects
@@
 			(project "SiganlGen"
 				(path "/e2db369b-fed9-4358-b449-15db5155edf2/76a7b521-7475-43f8-a5df-abb93f6b2174"
-					(reference "J3")
+					(reference "J4")
 					(unit 1)
 				)
@@
 		(on_board yes)
 		(dnp no)
-		(property "Reference" "J4"
+		(property "Reference" "J5"
 			(at 38.862 82.042 0)
 			(effects
@@
 			(project "SiganlGen"
 				(path "/e2db369b-fed9-4358-b449-15db5155edf2/76a7b521-7475-43f8-a5df-abb93f6b2174"
-					(reference "J4")
+					(reference "J5")
 					(unit 1)
 				)
@@
 		(on_board yes)
 		(dnp no)
-		(property "Reference" "J9"
+		(property "Reference" "J3"
 			(at 33.02 45.2121 0)
 			(effects
@@
 			(project "SiganlGen"
 				(path "/e2db369b-fed9-4358-b449-15db5155edf2/76a7b521-7475-43f8-a5df-abb93f6b2174"
-					(reference "J9")
-					(unit 1)
-				)
+					(reference "J3")
+					(unit 1)
+				)

Commit message: Final PCB version (probably)
Connections:
- net MUX2: now also J3.3 (Pin_3); no longer J3.4 (Pin_4)
- net MUX3: now also J3.4 (Pin_4); no longer J3.3 (Pin_3)
Changed lines of the file:
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@@
 	(hierarchical_label "MUX2"
 		(shape input)
-		(at 40.64 41.91 180)
+		(at 40.64 39.37 180)
 		(fields_autoplaced yes)
 		(effects
@@
 	(hierarchical_label "MUX3"
 		(shape input)
-		(at 40.64 39.37 180)
+		(at 40.64 41.91 180)
 		(fields_autoplaced yes)
 		(effects
