File: KiCad/SiganlGen.kicad_pcb (KiCad board)
At the start: 2 copper layers, 99.7 x 71.8 mm, 101 parts, among them J1 P_In, J2 Conn_Coaxial, J3 Btn_Matrix, J4 LCD_Conn, J5 Enc_Conn, J6 Btn&Led, J7 PWR, K1 Relay_SPST-NO, Q1 BD135, Q2 BD136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

Commit message: silkscreen art
Parts:
- added G***: LOGO, LOGO, F.Cu at (200.7, 93.3)
- added G***: LOGO, pictures:swim, F.Cu at (174.6, 36.2)
- added G***: LOGO, pictures:pwr, F.Cu at (168.3, 36.8)
- added REF**: WEEE-Logo_4.2x6mm_SilkScreen, Symbol:WEEE-Logo_4.2x6mm_SilkScreen, F.Cu at (139.7, 36.2)
- added REF**: ESD-Logo_6.6x6mm_SilkScreen, Symbol:ESD-Logo_6.6x6mm_SilkScreen, F.Cu at (146.7, 36.2)
- added REF**: KiCad-Logo_5mm_SilkScreen, Symbol:KiCad-Logo_5mm_SilkScreen, F.Cu at (157.5, 36.8)
- moved J4 0.63 mm to (172.1, 91.4)
- moved J5 0.63 mm to (172.1, 78.7)
- moved J6 0.63 mm to (172.1, 61.0)
- moved J7 0.63 mm to (172.1, 54.6)
Routing:
- net +3V3: track 6.80 -> 6.17 mm
- net /UI.OUT1: track 6.24 -> 5.61 mm
- net /UI.IN0: track 6.24 -> 5.61 mm
- net /LCD.SDA: track 6.96 -> 6.33 mm
- net /LCD.SCL: track 7.37 -> 6.74 mm
- net /ENC.SW: track 6.24 -> 5.61 mm
- net /ENC.DT: track 6.24 -> 5.61 mm
- net /ENC.CLK: track 6.24 -> 5.61 mm
- net +5V: track 87.6 -> 88.3 mm
- net GND: vias 439 -> 463
Other:
- board text added: "12V/1A"
- board text added: "BC(263671) WR(263607) Pico_Signal_Generator PWr PGr: EKA 23/24"
- board text added: "JLCJLCJLCJLC"
- board text added: "We don't make errors, we have happy syntax accidents; ~Bob Ross {dblquote}The Joy of Electronics{dblquote}"
